Commit message: Update my_rb1_robot.urdf

File: my_rb1_description/urdf/my_rb1_robot.urdf (robot description, URDF)
Before this commit: robot my_rb1_robot, 7 links, 6 joints
Links:
- link back_caster: geometry collision sphere radius=0.025; collision sphere radius=0.05
- link front_caster: geometry collision sphere radius=0.025; collision sphere radius=0.05
